File: 32X_main1.kicad_sch (KiCad schematic)
At the start: 27 parts, among them IC504 315-5818, IC505 315-5805, IC509 74AC04

Commit message: update readme, update kicad version, add connection between 81 and GND
Changed lines of the file:
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@@
 (kicad_sch
-	(version 20231120)
+	(version 20250114)
 	(generator "eeschema")
-	(generator_version "8.0")
+	(generator_version "9.0")
 	(paper "A3")
 	(title_block
@@
 		(comment 1 "Neptune")
 	)
+	(rectangle
+		(start 40.64 45.72)
+		(end 103.505 142.24)
+		(stroke
+			(width 0)
+			(type dash)
+		)
+		(fill
+			(type none)
+		)
+	)
+	(text "(Bridge for other)"
+		(exclude_from_sim no)
+		(at 109.855 193.675 0)
+		(effects
+			(font
+				(size 1.27 1.27)
+			)
+			(justify left bottom)
+		)
+	)
+	(text "VA1 ONLY"
+		(exclude_from_sim no)
+		(at 91.44 49.53 0)
+		(effects
+			(font
+				(size 1.27 1.27)
+			)
+			(justify left bottom)
+		)
+	)
+	(text "THT bodges on later 32X main\nboards with SCA chip. If your\ndonor has this, CUT THE TRACE\nbefore installing the diode here.\nOtherwise leave bridge intact."
+		(exclude_from_sim no)
+		(at 97.79 179.07 0)
+		(effects
+			(font
+				(size 1.27 1.27)
+			)
+			(justify left bottom)
+		)
+	)
 	(junction
 		(at 96.52 99.06)
@@
 		)
 	)
-	(rectangle
-		(start 40.64 45.72)
-		(end 103.505 142.24)
-		(stroke
-			(width 0)
-			(type dash)
-		)
-		(fill
-			(type none)
-		)
-	)
-	(text "(Bridge for other)"
-		(exclude_from_sim no)
-		(at 109.855 193.675 0)
-		(effects
-			(font
-				(size 1.27 1.27)
-			)
-			(justify left bottom)
-		)
-	)
-	(text "VA1 ONLY"
-		(exclude_from_sim no)
-		(at 91.44 49.53 0)
-		(effects
-			(font
-				(size 1.27 1.27)
-			)
-			(justify left bottom)
-		)
-	)
-	(text "THT bodges on later 32X main\nboards with SCA chip. If your\ndonor has this, CUT THE TRACE\nbefore installing the diode here.\nOtherwise leave bridge intact."
-		(exclude_from_sim no)
-		(at 97.79 179.07 0)
-		(effects
-			(font
-				(size 1.27 1.27)
-			)
-			(justify left bottom)
-		)
-	)
