File: 32X_sub.kicad_sch (KiCad schematic)
At the start: 105 parts, among them IC511 315-5684, IC512 315-5788, IC515 74HC74, IC516 74LS00, T520 TestPoint, T526 TestPoint, T527 TestPoint, T528 TestPoint, T547 TestPoint, T548 TestPoint, T555 TestPoint, T599 AS, X501 *3

Commit message: update readme, update kicad version, add connection between 81 and GND
Changed lines of the file:
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@@
 (kicad_sch
-	(version 20231120)
+	(version 20250114)
 	(generator "eeschema")
-	(generator_version "8.0")
+	(generator_version "9.0")
 	(paper "A3")
 	(title_block
@@
 		(comment 1 "Neptune")
 	)
+	(rectangle
+		(start 249.555 255.27)
+		(end 297.18 279.4)
+		(stroke
+			(width 0)
+			(type default)
+		)
+		(fill
+			(type none)
+		)
+	)
+	(text "PAL"
+		(exclude_from_sim no)
+		(at 280.67 258.445 0)
+		(effects
+			(font
+				(size 1.27 1.27)
+				(bold yes)
+			)
+			(justify left bottom)
+		)
+	)
+	(text "*"
+		(exclude_from_sim no)
+		(at 251.46 258.445 0)
+		(effects
+			(font
+				(size 1.27 1.27)
+				(thickness 0.254)
+				(bold yes)
+			)
+			(justify left bottom)
+		)
+	)
+	(text "L604\nL605\nX501\nR540\nR541\nC570\nC574\nC575\nC578"
+		(exclude_from_sim no)
+		(at 257.175 278.13 0)
+		(effects
+			(font
+				(size 1.27 1.27)
+			)
+			(justify left bottom)
+		)
+	)
+	(text "NTSC"
+		(exclude_from_sim no)
+		(at 265.43 258.445 0)
+		(effects
+			(font
+				(size 1.27 1.27)
+				(bold yes)
+			)
+			(justify left bottom)
+		)
+	)
+	(text "10uH\n82uH\n4.43361875MHz\n430\n680\n68pF\n15pF\n47pF\n82pF"
+		(exclude_from_sim no)
+		(at 280.67 278.13 0)
+		(effects
+			(font
+				(size 1.27 1.27)
+			)
+			(justify left bottom)
+		)
+	)
+	(text "1\n2\n3\n4\n5\n8\n9\n10\n11"
+		(exclude_from_sim no)
+		(at 251.46 278.13 0)
+		(effects
+			(font
+				(size 1.27 1.27)
+			)
+			(justify left bottom)
+		)
+	)
+	(text "12uH\n100uH\n3.579545MHz\n560\n1.2K\n47pF\n18pF\n56pF\n100pF"
+		(exclude_from_sim no)
+		(at 265.43 278.13 0)
+		(effects
+			(font
+				(size 1.27 1.27)
+			)
+			(justify left bottom)
+		)
+	)
+	(text "REF"
+		(exclude_from_sim no)
+		(at 257.175 258.445 0)
+		(effects
+			(font
+				(size 1.27 1.27)
+				(bold yes)
+			)
+			(justify left bottom)
+		)
+	)
+	(text "Bridged, cut and place\na cap if required"
+		(exclude_from_sim no)
+		(at 323.85 80.01 0)
+		(effects
+			(font
+				(size 1.27 1.27)
+			)
+			(justify left bottom)
+		)
+	)
 	(junction
 		(at 152.4 33.02)
@@
 		)
 	)
-	(rectangle
-		(start 249.555 255.27)
-		(end 297.18 279.4)
-		(stroke
-			(width 0)
-			(type default)
-		)
-		(fill
-			(type none)
-		)
-	)
-	(text "PAL"
-		(exclude_from_sim no)
-		(at 280.67 258.445 0)
-		(effects
-			(font
-				(size 1.27 1.27)
-				(bold yes)
-			)
-			(justify left bottom)
-		)
-	)
-	(text "*"
-		(exclude_from_sim no)
-		(at 251.46 258.445 0)
-		(effects
-			(font
-				(size 1.27 1.27)
-				(thickness 0.254)
-				(bold yes)
-			)
-			(justify left bottom)
-		)
-	)
-	(text "L604\nL605\nX501\nR540\nR541\nC570\nC574\nC575\nC578"
-		(exclude_from_sim no)
-		(at 257.175 278.13 0)
-		(effects
-			(font
-				(size 1.27 1.27)
-			)
-			(justify left bottom)
-		)
-	)
-	(text "NTSC"
-		(exclude_from_sim no)
-		(at 265.43 258.445 0)
-		(effects
-			(font
-				(size 1.27 1.27)
-				(bold yes)
-			)
-			(justify left bottom)
-		)
-	)
-	(text "10uH\n82uH\n4.43361875MHz\n430\n680\n68pF\n15pF\n47pF\n82pF"
-		(exclude_from_sim no)
-		(at 280.67 278.13 0)
-		(effects
-			(font
-				(size 1.27 1.27)
-			)
-			(justify left bottom)
-		)
-	)
-	(text "1\n2\n3\n4\n5\n8\n9\n10\n11"
-		(exclude_from_sim no)
-		(at 251.46 278.13 0)
-		(effects
-			(font
-				(size 1.27 1.27)
-			)
-			(justify left bottom)
-		)
-	)
-	(text "12uH\n100uH\n3.579545MHz\n560\n1.2K\n47pF\n18pF\n56pF\n100pF"
-		(exclude_from_sim no)
-		(at 265.43 278.13 0)
-		(effects
-			(font
-				(size 1.27 1.27)
-			)
-			(justify left bottom)
-		)
-	)
-	(text "REF"
-		(exclude_from_sim no)
-		(at 257.175 258.445 0)
-		(effects
-			(font
-				(size 1.27 1.27)
-				(bold yes)
-			)
-			(justify left bottom)
-		)
-	)
-	(text "Bridged, cut and place\na cap if required"
-		(exclude_from_sim no)
-		(at 323.85 80.01 0)
-		(effects
-			(font
-				(size 1.27 1.27)
-			)
-			(justify left bottom)
-		)
-	)
